File: RCT-X-Logger.sch (KiCad schematic (older format))
At the start: 55 parts

Commit message: MountingHole追加
Parts:
- added H? (x4): MountingHole, symbol Mechanical:MountingHole
Changed lines of the file:
@@
 Wire Wire Line
 	10050 5000 9300 5000
+$Comp
+L Mechanical:MountingHole H?
+U 1 1 5E55EC07
+P 1200 6850
+F 0 "H?" H 1300 6896 50  0000 L CNN
+F 1 "MountingHole" H 1300 6805 50  0000 L CNN
+F 2 "" H 1200 6850 50  0001 C CNN
+F 3 "~" H 1200 6850 50  0001 C CNN
+	1    1200 6850
+	1    0    0    -1
+$EndComp
+$Comp
+L Mechanical:MountingHole H?
+U 1 1 5E5603B3
+P 1200 7100
+F 0 "H?" H 1300 7146 50  0000 L CNN
+F 1 "MountingHole" H 1300 7055 50  0000 L CNN
+F 2 "" H 1200 7100 50  0001 C CNN
+F 3 "~" H 1200 7100 50  0001 C CNN
+	1    1200 7100
+	1    0    0    -1
+$EndComp
+$Comp
+L Mechanical:MountingHole H?
+U 1 1 5E560636
+P 1200 7350
+F 0 "H?" H 1300 7396 50  0000 L CNN
+F 1 "MountingHole" H 1300 7305 50  0000 L CNN
+F 2 "" H 1200 7350 50  0001 C CNN
+F 3 "~" H 1200 7350 50  0001 C CNN
+	1    1200 7350
+	1    0    0    -1
+$EndComp
+$Comp
+L Mechanical:MountingHole H?
+U 1 1 5E560A57
+P 1200 7600
+F 0 "H?" H 1300 7646 50  0000 L CNN
+F 1 "MountingHole" H 1300 7555 50  0000 L CNN
+F 2 "" H 1200 7600 50  0001 C CNN
+F 3 "~" H 1200 7600 50  0001 C CNN
+	1    1200 7600
+	1    0    0    -1
+$EndComp
 $EndSCHEMATC

Commit message: [update] 回路初版完成, 部品決定
Parts:
- removed C?: 47uF, symbol Device:C
- removed U?: CY8C5868LTI-LP039, symbol KUTKiCad_symbol:CY8C5868LTI-LP039
- added R? (x4): 4.7kΩ, Resistor_SMD:R_0402_1005Metric, symbol Device:R
- added R? (x4): 22Ω, Resistor_SMD:R_0402_1005Metric, symbol Device:R
- added U5: CY8C58xxLTI-LPxxx, KUTKiCad_footprint:Cypress_QFN-68_EP_8x8_Pitch0.4mm, symbol KUTKiCad_symbol:CY8C58xxLTI-LPxxx
- BT1: renamed from BT?; footprint (none) -> Battery:BatteryHolder_Seiko_MS621F; Agency (none) -> Chip1stop; MPN (none) -> MS621FE; Manufacture (none) -> Seiko Instrument
- C1, C2, C5, C6: renamed from C?; footprint (none) -> Capacitor_SMD:C_0603_1608Metric; Agency (none) -> Digikey; MPN (none) -> GRM188R61E106MA73D; Manufacture (none) -> muRata; Value (none) -> 10uF
- C10, C11, C12, C13, C15, C24, C25, C26, C4, C8, C9: renamed from C?; footprint (none) -> Capacitor_SMD:C_0603_1608Metric; Agency (none) -> Digikey; MPN (none) -> GRM188R72A104KA35D
- C14, C16, C17, C18: renamed from C?; footprint (none) -> Capacitor_SMD:C_0402_1005Metric; Agency (none) -> Digikey; MPN (none) -> GRM155R61E105KA12D
- C19, C20, C21, C22: renamed from C?; value C -> 9pF; footprint (none) -> Capacitor_SMD:C_0201_0603Metric; Agency (none) -> Digikey; MPN (none) -> GRM0335C1E9R0CA01D
- C23: renamed from C?; footprint (none) -> Capacitor_SMD:C_0603_1608Metric; Agency (none) -> Digikey; MPN (none) -> GRM185R61C475ME11D
- C3: renamed from C?; footprint (none) -> Capacitor_SMD:C_0402_1005Metric; Agency (none) -> Digikey; MPN (none) -> GRM155R71H472KA01D; Manufacture (none) -> muRata; Value (none) -> 4700pF
- C7: renamed from C?; value 10uF -> 0.1uF; footprint (none) -> Capacitor_SMD:C_0603_1608Metric; Agency (none) -> Digikey; MPN (none) -> GRM188R72A104KA35D
- D1: renamed from D?; value LED -> LED_BLUE; footprint (none) -> LED_SMD:LED_0603_1608Metric; MPN (none) -> SMLE12BC7TT86
- D2: renamed from D?; value LED -> LED_OR; footprint (none) -> LED_SMD:LED_0603_1608Metric; MPN (none) -> SML-E12D8WT86
- D3: renamed from D?; footprint (none) -> KUTKiCad_footprint:D_SOD-723; Agency (none) -> Digikey; MPN (none) -> 1SS400GT2R
- H1, H2, H3, H4: renamed from H?; footprint (none) -> MountingHole:MountingHole_3.5mm
- J1: renamed from J?; footprint (none) -> KUTKiCad_footprint:Hirose_ZX_ZX62D-B-5P8; Agency (none) -> Digikey; MPN (none) -> ZX62D-B-5P8(30)
- P1: renamed from P?; footprint (none) -> KUTKiCad_footprint:JST_JQ_05JQ-BT_1x05_P2.5mm_Vertical; Agency (none) -> Digikey; MPN (none) -> 05JQ-BT
- R1, R2: renamed from R?; footprint (none) -> Resistor_SMD:R_0402_1005Metric; Agency (none) -> Digikey; MPN (none) -> ERJ-2GEJ560X
- R10, R9: renamed from R?; footprint (none) -> Resistor_SMD:R_0402_1005Metric; Agency (none) -> Digikey; MPN (none) -> ERJ-2GEJ472X
- R11: renamed from R?; footprint (none) -> Resistor_SMD:R_0402_1005Metric; Agency (none) -> Digikey; MPN (none) -> ERJ-2GEJ683X
- R3, R4: renamed from R?; footprint (none) -> Resistor_SMD:R_0402_1005Metric; Agency (none) -> Digikey; MPN (none) -> ERJ-2GEJ220X
- R5, R6, R7, R8: renamed from R?; footprint (none) -> Resistor_SMD:R_0402_1005Metric; Agency (none) -> Digikey; MPN (none) -> ERJ-2GEJ221X
- U1: renamed from U?; footprint (none) -> KUTKiCad_footprint:JST_XH_S4B-XH-SM4-TB_1x04_P2.5mm; Agency (none) -> chip1stop; MPN (none) -> S4B-XH-SM4-TB
- U2: renamed from U?; Agency (none) -> Digikey; MPN (none) -> LT1761MPS5-5#TRMPBF
- U3: renamed from U?; footprint (none) -> Package_DFN_QFN:DFN-8-1EP_3x3mm_P0.5mm_EP1.66x2.38mm; Agency (none) -> Digikey; MPN (none) -> LT1965EDD-3.3#PBF
- U4: renamed from U?; footprint (none) -> Package_DFN_QFN:DFN-8-1EP_3x3mm_P0.65mm_EP1.55x2.4mm; Agency (none) -> Digikey; MPN (none) -> NCV7342MW3R2G
- U6: renamed from U?; value CAM-M8 -> CAM-M8C; footprint (none) -> KUTKiCad_footprint:ublox-CAM; Agency (none) -> Digikey; MPN (none) -> CAM-M8C-0-10
- U7: renamed from U?; footprint (none) -> KUTKiCad_footprint:TE_Sensor_MS8607; Agency (none) -> Digikey; MPN (none) -> MS560702BA03-50
- U8: renamed from U?; Agency (none) -> Digikey; MPN (none) -> W25N01GVZEIG TR
- U9: renamed from U?; footprint (none) -> Package_DFN_QFN:DFN-6-1EP_3x3mm_P1mm_EP1.5x2.4mm; Agency (none) -> Digikey; MPN (none) -> HPP845E131R4
- Y1: renamed from Y?; value Crystal -> Crystal_kHz; Agency (none) -> Digikey; MPN (none) -> FC-135R 32.7680KF-AC3
- Y2: renamed from Y?; value Crystal -> Crystal_MHz
Connections:
- net +3V3: now also R?.2, R?.2, R?.2, R?.2, U5.17 (VDDIO1), U5.24 (VDDD), U5.35 (VDDIO3), U5.44 (VDDA), U5.52 (VDDIO0), U5.59 (VDDD), U5.67 (VDDIO2)
- net CAN-RXD: now also U5.2 (P2[7])
- net CAN-STB: now also U5.68 (P2[5])
- net CAN-TXD: now also U5.1 (P2[6])
- net Flash-MISO: now also R?.2, U5.62 (P2[0]); no longer U8.2 (DO)
- net Flash-MOSI: now also R?.2, U5.63 (P2[1]); no longer U8.5 (DI)
- net Flash-SCLK: now also R?.2, U5.64 (P2[2]); no longer U8.6 (CLK)
- net Flash-~CS: now also R?.2, U5.65 (P2[3]); no longer U8.1 (~CS)
- net GND: now also C20.1, U5.25 (VSSD), U5.43 (VSSA), U5.45 (VSSD), U5.5 (VSSB), U5.58 (VSSD), U5.6 (IND), U5.69 (PAD), U5.7 (VBOOST), U5.8 (VBAT), U5.9 (VSSD)
- net GNSS-1PPS: now also U5.32 (P3[3]/OA3P)
- net GNSS-RXD: now also U5.30 (P3[1]/IDAC3)
- net GNSS-TXD: now also U5.29 (P3[0]/IDAC1)
- net GNSS-~RESET: now also U5.31 (P3[2]/OA3N/REF1)
- net H-SCL: now also U5.51 (P0[3]/OA0N/REF0)
- net H-SDA: now also U5.50 (P0[2]/OA0P/SAR1REF)
- net PT-MISO: now also U5.53 (P0[4]/OA2P/SAR0REF)
- net PT-MOSI: now also U5.54 (P0[5]/OA2N)
- net PT-SCLK: now also U5.55 (P0[6]/IDAC0)
- net PT-~CS: now also U5.56 (P0[7]/IDAC2)
- net at U1.3 (CANH), U4.7 (CANH): now also R1.2; no longer R1.1
- net at U8.3 (~WP): now also R?.1
- net at U8.7 (~HOLD): now also R?.1
- net at P1.3 (XRES): now also U5.10 (XRES)
- net at P1.5 (SDAT): now also U5.11 (P1[0]/SWDIO/TMS)
- net at P1.4 (SCLK): now also U5.12 (P1[1]/SWDCK/TCK)
- net at R3.2: now also U5.22 (P15[6]/USB_DP)
- net at R4.2: now also U5.23 (P15[7]/USB_DN)
- net at C18.1: now also U5.26 (VCCD), U5.57 (VCCD)
- net at C22.2, Y2.2: now also U5.27 (P15[0]/MHzXTAL_XO)
- net at C21.2, Y2.1: now also U5.28 (P15[1]/MHzXTAL_XI)
- net at D1.1 (K): now also U5.3 (P12[4]/SIO)
- net at D2.1 (K): now also U5.4 (P12[5]/SIO)
- net at C20.2, Y1.2: now also U5.40 (P15[2]/kHzXTAL_XO)
- net at C19.2, Y1.1: now also U5.41 (P15[3]/kHzXTAL_XI)
- net at C17.1: now also U5.42 (VCCA)
- net at C3.1, R2.2: now also R1.1; no longer R1.2
- new net: R?.1, R?.1, U8.1 (~CS)
- new net: R?.1, R?.1, U8.2 (DO)
- new net: R?.1, U8.5 (DI)
- new net: R?.1, U8.6 (CLK)
- no-connect marks 33 -> 31
Other:
- moved on the sheet: BT1, C1, C10, C11, C12, C13, C14, C15, C16, C17, C18, C19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

Commit message: [update] 部品追記
Parts:
- U8: footprint (none) -> KUTKiCad_footprint:WSON-8_8x6mm_P1.27mm
- Y1: footprint (none) -> KUTKiCad_footprint:Crystal_SeikoEpson_FC-135
- Y2: footprint (none) -> Crystal:Crystal_SMD_SeikoEpson_TSX3225-4Pin_3.2x2.5mm; MPN (none) -> TSX-3225 24.0000MF15X-AC6
- gave numbers to parts that had none: 8
- renumbered R9 to R15, R10 to R17, R11 to R19
Other:
- moved on the sheet: BT1, C1, C10, C11, C12, C13, C14, C15, C16, C17, C18, C19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

Commit message: アートワークに合わせて配線変更
Parts:
- C10, C11, C12, C13, C15, C24, C25, C26, C4, C7, C8, C9: footprint Capacitor_SMD:C_0603_1608Metric -> Capacitor_SMD:C_0402_1005Metric; MPN GRM188R72A104KA35D -> GRM155R62A104KE14D
- U1: footprint KUTKiCad_footprint:JST_XH_S4B-XH-SM4-TB_1x04_P2.5mm -> Connector_JST:JST_XH_S4B-XH-A_1x04_P2.50mm_Horizontal; MPN S4B-XH-SM4-TB -> S4B-XH-A
- Y2: footprint Crystal:Crystal_SMD_SeikoEpson_TSX3225-4Pin_3.2x2.5mm -> KUTKiCad_footprint:Crystal_Murata_XRCHA; MPN TSX-3225 24.0000MF15X-AC6 -> XRCHA24M000F0A01R0
Connections:
- net Flash-MISO: now also U5.15 (P1[4]/TDI); no longer U5.62 (P2[0])
- net Flash-MOSI: now also U5.14 (P1[3]/SWV/TDO); no longer U5.63 (P2[1])
- net Flash-SCLK: now also U5.13 (P1[2]); no longer U5.64 (P2[2])
- net Flash-~CS: now also U5.16 (P1[5]/NTRST); no longer U5.65 (P2[3])
- net GND: no longer J1.6 (Shield)
- net GNSS-1PPS: now also U5.56 (P0[7]/IDAC2); no longer U5.32 (P3[3]/OA3P)
- net GNSS-RXD: now also U5.54 (P0[5]/OA2N); no longer U5.30 (P3[1]/IDAC3)
- net GNSS-TXD: now also U5.53 (P0[4]/OA2P/SAR0REF); no longer U5.29 (P3[0]/IDAC1)
- net GNSS-~RESET: now also U5.55 (P0[6]/IDAC0); no longer U5.31 (P3[2]/OA3N/REF1)
- net PT-MISO: now also U5.64 (P2[2]); no longer U5.53 (P0[4]/OA2P/SAR0REF)
- net PT-MOSI: now also U5.63 (P2[1]); no longer U5.54 (P0[5]/OA2N)
- net PT-SCLK: now also U5.62 (P2[0]); no longer U5.55 (P0[6]/IDAC0)
- net PT-~CS: now also U5.65 (P2[3]); no longer U5.56 (P0[7]/IDAC2)
- net at U5.3 (P12[4]/SIO): no longer D1.1 (K)
- net at U5.33 (P3[4]/OA1N): now also D1.1 (K)
- net at U5.34 (P3[5]/OA1P): now also D2.1 (K)
- net at U5.4 (P12[5]/SIO): no longer D2.1 (K)
- no-connect marks 31 -> 32
Other:
- moved on the sheet: D1, D2, P1, R5, R6
