File: RCT-X-Logger.sch (KiCad schematic (older format))
At the start: 66 parts, among them J1 USB_B_Micro, P1 KRC_Conn_SWD, U1 KRC_Conn_CAN, U2 LT1761-5, U3 LT1965xDD-3.3, U4 NCV7342, U5 CY8C58xxLTI-LPxxx, U6 CAM-M8C, U7 MS5607, U8 W25N01GVxxIG-IT, U9 HTU21D, Y1 Crystal_kHz, Y2 Crystal_MHz

Commit message: Completed Rev2
Parts:
- removed D1: LED_BLUE, LED_SMD:LED_0603_1608Metric, symbol Device:LED
- removed D2: LED_OR, LED_SMD:LED_0603_1608Metric, symbol Device:LED
- removed U7: MS5607, KUTKiCad_footprint:TE_Sensor_MS8607, symbol KUTKiCad_symbol:MS5607
- added D1: LED_RGBA, KUTKiCad_footprint:LED_LiteOn_LTST-C19HE1WT, symbol Device:LED_RGBA
- added F1: Polyfuse, Fuse:Fuse_0805_2012Metric, symbol Device:Polyfuse
- added J2: Conn_01x02, Connector_JST:JST_XH_B2B-XH-A_1x02_P2.50mm_Vertical, symbol Connector_Generic:Conn_01x02
- added R7: 820Ω, Resistor_SMD:R_0402_1005Metric, symbol Device:R
- added U6: MS5611, KUTKiCad_footprint:TE_Sensor_MS8607, symbol KUTKiCad_symbol:MS5611
- H1, H2, H3, H4: footprint MountingHole:MountingHole_3.5mm -> MountingHole:MountingHole_3.2mm_M3
- R5: value 220Ω -> 1.5kΩ; MPN ERJ-2GEJ221X -> ERJ-2GEJ152X
- R6: value 220Ω -> 820Ω; MPN ERJ-2GEJ221X -> ERJ-2GEJ821X
- R8: renamed from R7; value 220Ω -> 22Ω; MPN ERJ-2GEJ221X -> ERJ-2GEJ220X
- R9: renamed from R8; value 220Ω -> 22Ω; MPN ERJ-2GEJ221X -> ERJ-2GEJ220X
- U1: Agency chip1stop -> Digikey
- Y2: Agency (none) -> Digikey
- renumbered D3 to D2, R9 to R10, R10 to R11, R11 to R12, R12 to R13, R15 to R14, R13 to R15, R17 to R16, R14 to R17, R16 to R18, R18 to R19, R19 to R20, U6 to U7, U9 to U8, U8 to U9
Connections:
- net +3V3: now also D1.4 (A), U6.1 (VDD); no longer R5.2, R6.2
- net GND: now also U3.9 (PAD), U4.9 (PAD), U8.7 (PAD), U9.9 (PAD), J2.1 (Pin_1), U6.2 (PS), U6.3 (GND)
- net GNSS-1PPS: now also J2.2 (Pin_2)
- net PT-MISO: now also U6.6 (SDO)
- net PT-MOSI: now also U6.7 (SDI/SDA)
- net PT-SCLK: now also U6.8 (SCL/SCLK)
- net PT-~CS: now also U6.4 (CSB), U6.5 (CSB)
- net at C1.1, C2.1, U2.1 (VIN)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: now also F1.1; no longer U1.2 (VCC)
- net at U5.32 (P3[3]/OA3P): now also R5.1
- net at U5.33 (P3[4]/OA1N): now also R6.1
- net at U5.34 (P3[5]/OA1P): now also R7.1
- new net: F1.2, U1.2 (VCC)
- new net: D1.1 (RK), R5.2
- new net: D1.2 (GK), R6.2
- new net: D1.3 (BK), R7.2
- no-connect marks 32 -> 31
Other:
- moved on the sheet: BT1, C19, C20, C21, C22, C23, C24, C25, C26, C4, C7, D2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
